File: hardware/v2.0/R2R-DAC.kicad_sch (KiCad schematic)
At the start: 28 parts, among them U6 74LVC245A

Commit message: progress
Parts:
- renumbered C16 to C1, C17 to C2, R81 to R1, R90 to R10, R91 to R11, R92 to R12, R93 to R13, R94 to R14, R95 to R15, R96 to R16, R97 to R17, R98 to R18, R99 to R19, R82 to R2, R100 to R20, R101 to R21, R102 to R22, R103 to R23, R104 to R24, R105 to R25, R83 to R3, R84 to R4, R85 to R5, R86 to R6, R87 to R7, R88 to R8, R89 to R9, U6 to U3
