File: hardware/v2.0/iCE40HX-expansion.kicad_sch (KiCad schematic)
At the start: 48 parts, among them J1 EXT3, J2 EXT1, J3 AudioJack4, J4 Conn_01x34, J6 Conn_01x04, J7 Conn_02x10_Odd_Even, J8 DE15_Plug_HighDensity, J9 AudioJack4, U1 ADV7180BCP32Z-RL, U2 AMS1117-1.8, U5 74LVC245A, Y1 28.63636MHz

Commit message: progress
Parts:
- removed C1, C10, C12, C14, C24, C26, C28, C4, C5, C8: 0.1uf, Capacitor_SMD:C_0603_1608Metric, symbol Device:C_Small
- removed C11, C13, C15, C29, C6, C9: 10nf, Capacitor_SMD:C_0603_1608Metric, symbol Device:C_Small
- removed C2, C3: 47pf, Capacitor_SMD:C_0603_1608Metric, symbol Device:C_Small
- removed C22, C23, C25, C27: 10uf, Capacitor_SMD:C_0805_2012Metric, symbol Device:C_Small
- removed C7: 82nf, Capacitor_SMD:C_0603_1608Metric, symbol Device:C_Small
- removed J3, J9: AudioJack4, Connector_Audio:Jack_3.5mm_KoreanHropartsElec_PJ-320D-4A_Horizontal, symbol Connector_Audio:AudioJack4
- removed J6: Conn_01x04, Connector_PinHeader_2.54mm:PinHeader_1x04_P2.54mm_Vertical, symbol Connector_Generic:Conn_01x04
- removed J8: DE15_Plug_HighDensity, C711364:DSUB-TH_HYC06-HDR15B-060, symbol Connector:DE15_Plug_HighDensity
- removed R1, R4: 39, Resistor_SMD:R_0603_1608Metric, symbol Device:R_Small
- removed R2, R3: 36, Resistor_SMD:R_0603_1608Metric, symbol Device:R_Small
- removed R5: 1.69k, Resistor_SMD:R_0603_1608Metric, symbol Device:R_Small
- removed R56, R57: 270, Resistor_SMD:R_0603_1608Metric, symbol Device:R_Small
- removed R58: 0, Resistor_SMD:R_1206_3216Metric, symbol Device:R
- removed U1: ADV7180BCP32Z-RL, Package_CSP:LFCSP-32-1EP_5x5mm_P0.5mm_EP3.6x3.6mm, symbol C459884:ADV7180BCP32Z-RL
- removed U2: AMS1117-1.8, Package_TO_SOT_SMD:SOT-223-3_TabPin2, symbol Regulator_Linear:AMS1117-1.8
- removed U5: 74LVC245A, Package_SO:TSSOP-20_4.4x6.5mm_P0.65mm, symbol New_Library:74LVC245A
- removed Y1: 28.63636MHz, Crystal:Crystal_SMD_Abracon_ABM8AIG-4Pin_3.2x2.5mm, symbol Device:Crystal_GND24_Small
- added J3: EXT3, Connector_PinSocket_1.27mm:PinSocket_2x20_P1.27mm_Vertical_SMD, symbol Connector_Generic:Conn_02x20_Odd_Even
- added J5: EXT1, Connector_PinSocket_1.27mm:PinSocket_2x20_P1.27mm_Vertical_SMD, symbol Connector_Generic:Conn_02x20_Odd_Even
- added JP1: Jumper_2_Open, Jumper:SolderJumper-2_P1.3mm_Open_RoundedPad1.0x1.5mm, symbol Jumper:Jumper_2_Open
Connections:
- net +3V3: now also J3.5 (Pin_5)
- net +5V: now also J3.1 (Pin_1), JP1.1 (A); no longer J4.31 (Pin_31), J4.32 (Pin_32), J4.33 (Pin_33), J4.34 (Pin_34)
- net GND: now also J3.2 (Pin_2), J3.4 (Pin_4), J3.8 (Pin_8), J5.2 (Pin_2), J5.4 (Pin_4), J5.8 (Pin_8)
- net PIO0_00: no longer J7.17 (Pin_17)
- net PIO0_01: no longer J7.15 (Pin_15)
- net PIO0_02: no longer J7.13 (Pin_13)
- net PIO0_03: no longer J7.11 (Pin_11)
- net PIO0_04: no longer J7.9 (Pin_9)
- net PIO0_05: no longer J7.7 (Pin_7)
- net PIO0_06: no longer J7.5 (Pin_5)
- net PIO0_07: no longer J7.3 (Pin_3)
- net PIO0_08: no longer J7.1 (Pin_1)
- net PIO0_23: no longer J7.8 (Pin_8)
- net PIO0_24: no longer J7.6 (Pin_6)
- net PIO0_25: no longer J7.4 (Pin_4)
- net PIO0_26: no longer J7.2 (Pin_2)
- net PIO0_27: no longer J7.12 (Pin_12)
- net PIO0_28: no longer J7.14 (Pin_14)
- net PIO0_29: no longer J7.16 (Pin_16)
- net PIO0_30: no longer J7.18 (Pin_18)
- net PIO1_23: now also J4.6 (Pin_6); no longer J4.13 (Pin_13)
- net PIO1_24: now also J4.7 (Pin_7); no longer J4.12 (Pin_12)
- net PIO1_25: now also J4.8 (Pin_8); no longer J4.11 (Pin_11)
- net PIO1_26: now also J4.9 (Pin_9); no longer J4.10 (Pin_10)
- net PIO1_27: now also J4.10 (Pin_10); no longer J4.9 (Pin_9)
- net PIO1_28: now also J4.11 (Pin_11); no longer J4.8 (Pin_8)
- net PIO1_29: now also J4.12 (Pin_12); no longer J4.7 (Pin_7)
- net PIO1_30: now also J4.13 (Pin_13); no longer J4.6 (Pin_6)
- net PIO1_31: now also J4.14 (Pin_14); no longer J4.21 (Pin_21)
- net PIO1_32: now also J4.15 (Pin_15); no longer J4.20 (Pin_20)
- net PIO1_33: now also J4.16 (Pin_16); no longer J4.19 (Pin_19)
- net PIO1_34: now also J4.17 (Pin_17); no longer J4.18 (Pin_18)
- net PIO1_35: now also J4.18 (Pin_18); no longer J4.17 (Pin_17)
- net PIO1_36: now also J4.19 (Pin_19); no longer J4.16 (Pin_16)
- net PIO1_37: now also J4.20 (Pin_20); no longer J4.15 (Pin_15)
- net PIO1_38: now also J4.21 (Pin_21); no longer J4.14 (Pin_14)
- net PIO1_39: now also J4.22 (Pin_22); no longer J4.29 (Pin_29)
- net PIO1_40: now also J4.23 (Pin_23); no longer J4.28 (Pin_28)
- net PIO1_41: now also J4.24 (Pin_24); no longer J4.27 (Pin_27)
- net PIO1_42: now also J4.25 (Pin_25); no longer J4.26 (Pin_26)
- net PIO1_43: now also J4.26 (Pin_26); no longer J4.25 (Pin_25)
- net PIO1_44: now also J4.27 (Pin_27); no longer J4.24 (Pin_24)
- net PIO1_45: now also J4.28 (Pin_28); no longer J4.23 (Pin_23)
- net PIO1_46: now also J4.29 (Pin_29); no longer J4.22 (Pin_22)
- new net: J4.31 (Pin_31), J4.32 (Pin_32), J4.33 (Pin_33), J4.34 (Pin_34), JP1.2 (B)
- no-connect marks 15 -> 30
Other:
- removed sheet R2R-DAC
- removed sheet R2R-DAC1
- removed sheet R2R-DAC2
- added sheet VGA (VGA.kicad_sch)
- added sheet adv7611 (adv7611.kicad_sch)
- added sheet power (power.kicad_sch)
- added sheet tw884x (tw884x.kicad_sch)
- note added: "HDMI"
- note added: "LEDS"
- note added: "TW8847"
- note added: "VGA"
- note removed: "1V8 LDO"
- note removed: "ADDR = 40h"
- note removed: "DECODER"
- note removed: "EXTERNAL"
- note removed: "INDICATOR"
- note removed: "R2R DAC"
- note removed: "SYNC BUFFER"
- moved on the sheet: J1, J2, J4, J7
